File: SL_ADC_MCU_PCB.kicad_pcb (KiCad board)
At the start: 2 copper layers, 42 parts, among them IC1 ADS8528SPM, J1 Analog header, J2 GPIO breakpoints

Commit message: capacitors
Parts:
- C1, C18, C2, C3, C4, C5, C8: moved to B.Cu
- moved C18 90.2 mm to (110.2, 79.7), turned to 90 degrees
- moved C9 87.6 mm to (118.0, 99.0)
- moved C8 82.0 mm to (119.5, 87.0)
- moved C15 81.8 mm to (124.2, 86.2), turned to -90 degrees
- moved C5 78.5 mm to (111.0, 74.0), turned to 90 degrees
- moved C17 77.6 mm to (122.0, 70.7), turned to 90 degrees
- moved C12 74.8 mm to (119.0, 66.0), turned to 90 degrees
- moved C16 74.4 mm to (126.8, 74.7), turned to -90 degrees
- moved C1 73.9 mm to (118.5, 74.2), turned to 90 degrees
- moved C2 72.4 mm to (121.5, 81.5), turned to 180 degrees
- moved C11 70.8 mm to (124.2, 74.5), turned to 90 degrees
- moved C3 70.6 mm to (121.5, 79.0)
- moved C4 69.3 mm to (121.5, 77.0)
- moved C10 66.6 mm to (132.0, 83.0)
- moved C13 61.6 mm to (132.5, 74.0)
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Connections:
- IC1 pad 63: /CH_C1 -> /REFCP
Routing:
- net /AGND: track 0.00 -> 75.0 mm, vias 0 -> 7
- net /DB15: track 57.6 -> 0.00 mm, vias 1 -> 0
- net /AVDD: track 0.00 -> 31.0 mm, vias 0 -> 6
- net /REFN: track 0.00 -> 14.9 mm
- net /REFAP: track 0.00 -> 13.6 mm
- net /REFIO: track 0.00 -> 13.5 mm
- net /REFBP: track 0.00 -> 9.30 mm
- net /~PAR/SER: track 74.8 -> 82.8 mm
- net /~STBY: track 71.4 -> 79.0 mm
- net /REFEN/~WR: track 66.6 -> 74.1 mm
- net /RESET: track 72.3 -> 79.7 mm
- net /~RD: track 63.2 -> 70.3 mm
- net /~CS/~FS: track 60.4 -> 67.5 mm
- net /REFDP: track 0.00 -> 7.03 mm
- net /DVDD: track 0.00 -> 4.84 mm, vias 0 -> 1
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