File: SL_ADC_MCU_PCB.kicad_sch (KiCad schematic)
At the start: 22 parts, among them IC1 ADS8528SPM, J1 Conn_02x14_Counter_Clockwise

Commit message: added gpoi headers
Parts:
- added J2: Conn_02x08_Counter_Clockwise, Connector_PinHeader_2.54mm:PinHeader_2x08_P2.54mm_Vertical, symbol Connector_Generic:Conn_02x08_Counter_Clockwise
- added J3: Conn_02x16_Counter_Clockwise, Connector_PinHeader_2.54mm:PinHeader_2x16_P2.54mm_Vertical, symbol Connector_Generic:Conn_02x16_Counter_Clockwise
Connections:
- net ASLEEP: now also J3.19 (Pin_19)
- net BUSY/INT: now also J3.21 (Pin_21)
- net CONVST_A: now also J3.32 (Pin_32)
- net CONVST_B: now also J3.31 (Pin_31)
- net CONVST_C: now also J3.30 (Pin_30)
- net CONVST_D: now also J3.29 (Pin_29)
- net DB0: now also J3.1 (Pin_1)
- net DB1: now also J3.2 (Pin_2)
- net DB10: now also J3.11 (Pin_11)
- net DB11: now also J3.12 (Pin_12)
- net DB12: now also J3.13 (Pin_13)
- net DB13: now also J3.14 (Pin_14)
- net DB14: now also J3.15 (Pin_15)
- net DB15: now also J3.16 (Pin_16)
- net DB2: now also J3.3 (Pin_3)
- net DB3: now also J3.4 (Pin_4)
- net DB4: now also J3.5 (Pin_5)
- net DB5: now also J3.6 (Pin_6)
- net DB6: now also J3.7 (Pin_7)
- net DB7: now also J3.8 (Pin_8)
- net DB8: now also J3.9 (Pin_9)
- net DB9: now also J3.10 (Pin_10)
- net RANGE/XCLK: now also J3.22 (Pin_22)
- net RESET: now also J3.27 (Pin_27)
- net STM_D0: now reaches STM1.D0
- net STM_D0: now also J2.13 (Pin_13)
- net STM_D1: now reaches STM1.D1
- net STM_D1: now also J2.12 (Pin_12)
- net STM_D10: now reaches STM1.D10
- net STM_D10: now also J2.11 (Pin_11)
- net STM_D3: now reaches STM1.D3
- net STM_D3: now also J2.8 (Pin_8)
- net STM_D4: now reaches STM1.D4
- net STM_D4: now also J2.14 (Pin_14)
- net STM_D5: now reaches STM1.D5
- net STM_D5: now also J2.6 (Pin_6)
- net STM_D6: now reaches STM1.D6
- net STM_D6: now also J2.7 (Pin_7)
- net STM_D7: now reaches STM1.D7
- net STM_D7: now also J2.5 (Pin_5)
- net STM_D8: now reaches STM1.D8
- net STM_D8: now also J2.10 (Pin_10)
- net STM_D9: now reaches STM1.D9
- net STM_D9: now also J2.9 (Pin_9)
- net STM_E0: now reaches STM1.E0
- net STM_E0: now also J2.4 (Pin_4)
- net STM_E1: now reaches STM1.E1
- net STM_E1: now also J2.3 (Pin_3)
- net STM_E3: now reaches STM1.E3
- net STM_E3: now also J2.15 (Pin_15)
- net STM_E4: now reaches STM1.E4
- net STM_E4: now also J2.16 (Pin_16)
- net STM_E5: now reaches STM1.E5
- net STM_E5: now also J2.1 (Pin_1)
- net STM_E6: now reaches STM1.E6
- net STM_E6: now also J2.2 (Pin_2)
- new net -CS/-FS: J3.28 (Pin_28)
- new net -HW/SW: J3.20 (Pin_20)
- new net -PAR/SER: J3.23 (Pin_23)
- new net -RD: J3.26 (Pin_26)
- new net -STBY: J3.25 (Pin_25)
- new net REFEN/-WR: J3.24 (Pin_24)
Other:
- moved on the sheet: J1

Commit message: made a few visual edits and added a bunch of testpoints which apparently asks to 'annotate schematic' in the PCB editor, erm...
Parts:
- removed J3: Conn_02x16_Counter_Clockwise, Connector_PinHeader_2.54mm:PinHeader_2x16_P2.54mm_Vertical, symbol Connector_Generic:Conn_02x16_Counter_Clockwise
- added TP_BUSY, TP_CONVSTA, TP_CONVSTB, TP_CONVSTC, TP_CONVSTD, TP_DB0, TP_DB1, TP_DB10, TP_DB11, TP_DB2, TP_DB3, TP_DB4, TP_DB5, TP_DB6, TP_DB7, TP_DB8, TP_DB9, TP_RD, TP_WR: 5117, 5117:KEYSTONE_5117, symbol 5117:5117
- J1: value Conn_02x14_Counter_Clockwise -> Analog header
- J2: value Conn_02x08_Counter_Clockwise -> GPIO breakpoints
Connections:
- net -5V-HVSS: now also J1.11 (Pin_11), J1.12 (Pin_12); no longer J1.26 (Pin_26), J1.3 (Pin_3)
- net 5V-HVDD: now also J1.10 (Pin_10), J1.9 (Pin_9); no longer J1.2 (Pin_2), J1.27 (Pin_27)
- net AGND: now also J1.7 (Pin_7), J1.8 (Pin_8); no longer J1.23 (Pin_23), J1.24 (Pin_24)
- net AVDD: now also J1.2 (Pin_2); no longer J1.28 (Pin_28)
- net CH_A0: now also J1.27 (Pin_27), J1.28 (Pin_28); no longer J1.22 (Pin_22), J1.7 (Pin_7)
- net CH_A1: now also J1.25 (Pin_25), J1.26 (Pin_26); no longer J1.21 (Pin_21), J1.8 (Pin_8)
- net CH_B0: now also J1.23 (Pin_23), J1.24 (Pin_24); no longer J1.20 (Pin_20), J1.9 (Pin_9)
- net CH_B1: now also J1.21 (Pin_21), J1.22 (Pin_22); no longer J1.10 (Pin_10), J1.19 (Pin_19)
- net CH_C0: now also J1.19 (Pin_19), J1.20 (Pin_20); no longer J1.11 (Pin_11), J1.18 (Pin_18)
- net CH_C1: now also J1.18 (Pin_18); no longer J1.12 (Pin_12)
- net CH_D0: now also J1.15 (Pin_15); no longer J1.13 (Pin_13)
- net CH_D1: now also J1.13 (Pin_13); no longer J1.15 (Pin_15)
- net DVDD: now also J1.3 (Pin_3); no longer J1.25 (Pin_25)
Other:
- note added: "HEADERS"
- note added: "TESTPOINTS"
- moved on the sheet: J1, J2

Commit message: capacitors yet to route, rest done
Parts:
- renumbered TP_BUSY to TP_BUSY1, TP_CONVSTA to TP_CONVSTA1, TP_CONVSTB to TP_CONVSTB1, TP_CONVSTC to TP_CONVSTC1, TP_CONVSTD to TP_CONVSTD1, TP_RD to TP_RD1, TP_WR to TP_WR1
Changed lines of the file:
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@@
 		(dnp no)
 		(fields_autoplaced yes)
-		(property "Reference" "TP_CONVSTC"
+		(property "Reference" "TP_CONVSTC1"
 			(at 464.82 298.4499 0)
 			(effects
@@
 			(project "SL_ADC_MCU_PCB"
 				(path "/3f4eb23c-7a54-403d-a4d1-8d06ed1540f4"
-					(reference "TP_CONVSTC")
+					(reference "TP_CONVSTC1")
 					(unit 1)
 				)
@@
 		(dnp no)
 		(fields_autoplaced yes)
-		(property "Reference" "TP_CONVSTB"
+		(property "Reference" "TP_CONVSTB1"
 			(at 464.82 292.0999 0)
 			(effects
@@
 			(project "SL_ADC_MCU_PCB"
 				(path "/3f4eb23c-7a54-403d-a4d1-8d06ed1540f4"
-					(reference "TP_CONVSTB")
+					(reference "TP_CONVSTB1")
 					(unit 1)
 				)
@@
 		(dnp no)
 		(fields_autoplaced yes)
-		(property "Reference" "TP_WR"
+		(property "Reference" "TP_WR1"
 			(at 464.82 327.2853 0)
 			(effects
@@
 			(project "SL_ADC_MCU_PCB"
 				(path "/3f4eb23c-7a54-403d-a4d1-8d06ed1540f4"
-					(reference "TP_WR")
+					(reference "TP_WR1")
 					(unit 1)
 				)
@@
 		(dnp no)
 		(fields_autoplaced yes)
-		(property "Reference" "TP_CONVSTD"
+		(property "Reference" "TP_CONVSTD1"
 			(at 464.82 303.9045 0)
 			(effects
@@
 			(project "SL_ADC_MCU_PCB"
 				(path "/3f4eb23c-7a54-403d-a4d1-8d06ed1540f4"
-					(reference "TP_CONVSTD")
+					(reference "TP_CONVSTD1")
 					(unit 1)
 				)
@@
 		(dnp no)
 		(fields_autoplaced yes)
-		(property "Reference" "TP_RD"
+		(property "Reference" "TP_RD1"
 			(at 464.82 321.3099 0)
 			(effects
@@
 			(project "SL_ADC_MCU_PCB"
 				(path "/3f4eb23c-7a54-403d-a4d1-8d06ed1540f4"
-					(reference "TP_RD")
+					(reference "TP_RD1")
 					(unit 1)
 				)
@@
 		(dnp no)
 		(fields_autoplaced yes)
-		(property "Reference" "TP_BUSY"
+		(property "Reference" "TP_BUSY1"
 			(at 464.82 333.6353 0)
 			(effects
@@
 			(project "SL_ADC_MCU_PCB"
 				(path "/3f4eb23c-7a54-403d-a4d1-8d06ed1540f4"
-					(reference "TP_BUSY")
+					(reference "TP_BUSY1")
 					(unit 1)
 				)
@@
 		(dnp no)
 		(fields_autoplaced yes)
-		(property "Reference" "TP_CONVSTA"
+		(property "Reference" "TP_CONVSTA1"
 			(at 464.82 285.7499 0)
 			(effects
@@
 			(project "SL_ADC_MCU_PCB"
 				(path "/3f4eb23c-7a54-403d-a4d1-8d06ed1540f4"
-					(reference "TP_CONVSTA")
+					(reference "TP_CONVSTA1")
 					(unit 1)
 				)

Commit message: capacitors
Parts:
- STM1: value ~ -> (none)
Connections:
- net CH_C1: no longer IC1.63 (REFCP)
- net REFCP: now also IC1.63 (REFCP)
